Commit message: make inverse dynamics controller in 3dof single legged robot

File: camel-code-raisim/rsc/camel_single_leg_3dof.urdf (robot description, URDF)
Before this commit: robot camel_single_leg_bot_3dof, 6 links, 5 joints
Joints:
- joint linear_guide: origin xyz=0 -0.025 0.7 rpy=0 0 0 -> xyz=0 -0.025 0 rpy=0 0 0
