Commit message: Cubli PDcontroller get two verson whether they have trajectory generator

File: camel-code-raisim/rsc/camel_cubli.urdf (robot description, URDF)
Before this commit: robot camel_simple_pendulum, 4 links, 3 joints
Links:
- link motor: mass 1 -> 0.335; geometry visual cylinder length=0.02 radius=0.05; visual cylinder length=0.2 radius=0.5

Commit message: update cubli urdf and velocity plottiong

File: camel-code-raisim/rsc/camel_cubli.urdf (robot description, URDF)
Before this commit: robot camel_simple_pendulum, 4 links, 3 joints
Links:
- added link wheel-ball1, mass 1.0; visual sphere radius=0.015
- added link wheel-ball2, mass 1.0; visual sphere radius=0.015
- added link wheel-rod; visual box size=0.018 0.2 0.018
- link base: geometry visual cylinder length=0.02 radius=0.005
- link board: mass 1 -> 0.070; geometry collision box size=0.018 0.1458 0.1458; visual box size=0.018 0.1458 0.1458
- link motor: geometry visual cylinder length=0.0385 radius=0.0372
Joints:
- removed joint motor-roll
- added joint motor-fix: type fixed, parent board, child motor, origin xyz=-0.021 0.0 0.1031 rpy=0 0 0
- added joint wheel-1: type fixed, parent wheel-rod, child wheel-ball1, origin xyz=0.015 0.1 0.0 rpy=0 0 0
- added joint wheel-2: type fixed, parent wheel-rod, child wheel-ball2, origin xyz=0.015 -0.1 0.0 rpy=0 0 0
- added joint wheel-roll: type revolute, parent board, child wheel-rod, origin xyz=0.009 0 0.1031 rpy=0 0 0, axis 1 0 0
- joint base-roll: origin xyz=0 0 0.1 rpy=0 0 0 -> xyz=0 0 0.01275 rpy=0 0 0
